Commit message: Initial commit

File: urdf/chair.urdf (robot description, URDF)
Before this commit: robot robotic_chair, 12 links, 11 joints
Links:
- added link cliff_sensor_front, mass 0.01; collision box size=0.02 0.05 0.01; visual box size=0.02 0.05 0.01
- link base_footprint: geometry visual cylinder length=0.01 radius=0.35
Joints:
- added joint cliff_sensor_front_joint: type fixed, parent base_link, child cliff_sensor_front, origin xyz=0.30 0 -0.10
- joint camera_joint: origin xyz=0.32 0 0.35 -> xyz=0.32 0 0.25

Commit message: Add robotic_chair_description full content

File: urdf/chair.urdf (robot description, URDF)
Before this commit: robot robotic_chair, 13 links, 12 joints
Links:
- added link footrest_link, mass 0.5; collision box size=0.35 0.30 0.02; visual box size=0.35 0.30 0.02
- link backrest_link: geometry collision box size=0.05 0.45 0.35; visual box size=0.03 0.50 0.05
- link base_link: geometry collision box size=0.6 0.5 0.18; visual box size=0.05 0.55 0.16
- link left_wheel: geometry collision cylinder length=0.06 radius=0.16; visual cylinder length=0.03 radius=0.13
- link right_wheel: geometry collision cylinder length=0.06 radius=0.16; visual cylinder length=0.03 radius=0.13
- link seat_link: geometry collision box size=0.55 0.45 0.05; visual box size=0.04 0.04 0.20
Joints:
- added joint footrest_joint: type fixed, parent base_link, child footrest_link, origin xyz=0 0 -0.08
- joint front_left_caster_joint: origin xyz=0.25 0.20 -0.06 -> xyz=0.32 0.18 -0.07
- joint front_right_caster_joint: origin xyz=0.25 -0.20 -0.06 -> xyz=0.32 -0.18 -0.07
- joint left_wheel_joint: origin xyz=0 0.27 0.0 rpy=0 0 0 -> xyz=-0.05 0.30 0.0 rpy=0 0 0
- joint right_wheel_joint: origin xyz=0 -0.27 0.0 rpy=0 0 0 -> xyz=-0.05 -0.30 0.0 rpy=0 0 0
